Commit message: finish adding actuator, include wheel and caster

File: src/robot_description/urdf/fishbot/base.urdf.xacro (robot description, xacro)
@@ -13,4 +13,10 @@
             </visual>
         </link>
+        <link name="base_footprint" />
+        <joint name="base_joint" type="fixed">
+            <parent link="base_footprint" />
+            <child link="base_link" />
+            <origin xyz="0.0 0.0 ${length/2.0+0.032-0.001}" rpy="0 0 0" />
+        </joint>
     </xacro:macro>
 </robot>

File: src/robot_description/urdf/fishbot/fishbot.urdf.xacro (robot description, xacro)
@@ -11,3 +11,11 @@
     <xacro:laser_xacro xyz="0 0 0.1" />
     <xacro:camera_xacro xyz="0.1 0 0.075" />
+    <!-- 执行器组件 -->
+    <xacro:include filename="$(find robot_description)/urdf/fishbot/actuator/wheel.urdf.xacro" />
+    <xacro:include filename="$(find robot_description)/urdf/fishbot/actuator/caster.urdf.xacro" />
+    <!-- 执行器主动轮+从动轮 -->
+    <xacro:wheel_xacro wheel_name="left" xyz="0 0.10 -0.06" />
+    <xacro:wheel_xacro wheel_name="right" xyz="0 -0.10 -0.06 " />
+    <xacro:caster_xacro caster_name="front" xyz="0.08 0.0 -0.076" />
+    <xacro:caster_xacro caster_name="back" xyz="-0.08 0.0 -0.076" />
 </robot>
