Commit message: 通过编写urdf和xacro添加如下信息:
1. 传感器（激光雷达,相机和惯性测速）
2. 执行器（万向轮和驱动轮）
3. 物理属性（质量和惯性）
4. 两轮差速插件控制机器人
5. 在Gazebo中加载机器人模型,使用Gazebo标签扩展URDF
6. 创建xacro文件,并将gazebo文件保存为.world文件和.sdf文件

运行如下命令之后,可以实现gazebo中添加rviz中的模型
1. colcon build --packages-select robot_description
2. source install/setup.zsh
3. ros2 launch robot_description gazebo_sim.launch.py

可通过以下方式运行小车:
1. 可通过teleop_twist_keyboard来控制小车运行;
ros2 run teleop_twist_keyboard teleop_twist_keyboard

2. 直接通过命令行发布/cmd_vel话题;
ros2 topic pub /cmd_vel geometry_msgs/msg/Twist "{linear: {x: 1.0, y: 0.0, z: 0.0}, angular: {x: 0.0, y: 0.0, z: 0.5}}"

3. 直接通过代码发布/cmd_vel话题;
直接写python或C++代码,给话题/cmd_vel发布线速度和角速度

File: src/robot_description/urdf/fishbot/actuator/caster.urdf.xacro (robot description, xacro)
@@ -1,4 +1,5 @@
 <?xml version="1.0"?>
 <robot xmlns:xacro="http://www.ros.org/wiki/xacro">
+    <xacro:include filename="$(find robot_description)/urdf/fishbot/common_inertia.xacro" />
     <xacro:macro name="caster_xacro" params="caster_name xyz">
         <!--  声明一个万向轮的原点坐标、几何形状大小、材料颜色 -->
@@ -13,4 +14,14 @@
                 </material>
             </visual>
+            <collision>
+                <origin xyz="0 0 0" rpy="0 0 0" />
+                <geometry>
+                    <sphere radius="0.016" />
+                </geometry>
+                <material name="yellow">
+                    <color rgba="1.0 1.0 0.0 0.8" />
+                </material>
+            </collision>
+            <xacro:sphere_inertia m="0.01" r="0.016" />
         </link>
         <!-- 声明万向轮与本体的连接方式，origin和axis都以parent为基坐标 -->
@@ -22,4 +33,11 @@
             <axis xyz="0 0 0" />
         </joint>
+        <gazebo reference="${caster_name}_caster_link">
+            <mu1 value="0.0" />
+            <mu2 value="0.0" />
+            <kp value="1000000000.0" />
+            <kd value="1.0" />
+            <material>Gazebo/Yellow</material>
+        </gazebo>
     </xacro:macro>
 </robot>

File: src/robot_description/urdf/fishbot/actuator/wheel.urdf.xacro (robot description, xacro)
@@ -1,4 +1,5 @@
 <?xml version="1.0"?>
 <robot xmlns:xacro="http://www.ros.org/wiki/xacro">
+    <xacro:include filename="$(find robot_description)/urdf/fishbot/common_inertia.xacro" />
     <xacro:macro name="wheel_xacro" params="wheel_name xyz">
         <link name="${wheel_name}_wheel_link">
@@ -14,4 +15,16 @@
                 </material>
             </visual>
+            <collision>
+                <!-- 将r调整为90度，将轮子竖起来？这表示正确吗？ 是的， 竖起来的表示是正确的 -->
+                <!-- 此处，构建了原始的轮子样子 -->
+                <origin xyz="0 0 0" rpy="1.57079 0 0" />
+                <geometry>
+                    <cylinder length="0.04" radius="0.032" />
+                </geometry>
+                <material name="yellow">
+                    <color rgba="1.0 1.0 0.0 0.8" />
+                </material>
+            </collision>
+            <xacro:cylinder_inertia m="0.10" h="0.04" r="0.032" />
         </link>
         <!-- continuous 连续转动关节，对应轮子的旋转关节（主要指定旋转轴线），关节类型：固定和连续 -->
@@ -26,4 +39,15 @@
             <axis xyz="0 1 0" />
         </joint>
+        <gazebo reference="${wheel_name}_wheel_link">
+            <!-- 切向摩擦系数 -->
+            <mu1 value="20.0" />
+            <!-- 法向摩擦系数 -->
+            <mu2 value="20.0" />
+            <!--  刚度系数 -->
+            <kp value="1000000000.0" />
+            <!-- 阻尼系数 -->
+            <kd value="1.0" />
+            <material>Gazebo/Yellow</material>
+        </gazebo>
     </xacro:macro>
 </robot>

File: src/robot_description/urdf/fishbot/base.urdf.xacro (robot description, xacro)
@@ -1,4 +1,5 @@
 <?xml version="1.0"?>
 <robot xmlns:xacro="http://www.ros.org/wiki/xacro">
+    <xacro:include filename="$(find robot_description)/urdf/fishbot/common_inertia.xacro" />
     <xacro:macro name="base_xacro" params="length radius">
         <link name="base_link">
@@ -12,6 +13,20 @@
                 </material>
             </visual>
+            <collision>
+                <origin xyz="0 0 0" rpy="0 0 0" />
+                <geometry>
+                    <cylinder length="${length}" radius="${radius}" />
+                </geometry>
+                <material name="white">
+                    <color rgba="1.0 1.0 1.0 0.5" />
+                </material>
+            </collision>
+            <xacro:cylinder_inertia m="1.0" r="${radius}" h="${length}" />
         </link>
-        <link name="base_footprint" />
+        <link name="base_footprint">
+            <gazebo reference="base_footprint">
+                <static>false</static>  <!-- 静态模型会导致插件失效 -->
+            </gazebo>
+        </link>
         <joint name="base_joint" type="fixed">
             <parent link="base_footprint" />
@@ -19,4 +34,7 @@
             <origin xyz="0.0 0.0 ${length/2.0+0.032-0.001}" rpy="0 0 0" />
         </joint>
+        <gazebo reference="base_link">
+            <material>Gazebo/Gray</material>
+        </gazebo>
     </xacro:macro>
 </robot>

File: src/robot_description/urdf/fishbot/fishbot.urdf.xacro (robot description, xacro)
@@ -14,4 +14,6 @@
     <xacro:include filename="$(find robot_description)/urdf/fishbot/actuator/wheel.urdf.xacro" />
     <xacro:include filename="$(find robot_description)/urdf/fishbot/actuator/caster.urdf.xacro" />
+    <!-- Gazebo插件 -->
+    <xacro:include filename="$(find robot_description)/urdf/fishbot/plugins/gazebo_control_plugin.xacro" />
     <!-- 执行器主动轮+从动轮 -->
     <xacro:wheel_xacro wheel_name="left" xyz="0 0.10 -0.06" />
@@ -19,3 +21,4 @@
     <xacro:caster_xacro caster_name="front" xyz="0.08 0.0 -0.076" />
     <xacro:caster_xacro caster_name="back" xyz="-0.08 0.0 -0.076" />
+    <xacro:gazebo_control_plugin />
 </robot>

File: src/robot_description/urdf/fishbot/sensor/camera.urdf.xacro (robot description, xacro)
@@ -1,4 +1,5 @@
 <?xml version="1.0"?>
 <robot xmlns:xacro="http://www.ros.org/wiki/xacro">
+    <xacro:include filename="$(find robot_description)/urdf/fishbot/common_inertia.xacro" />
     <xacro:macro name="camera_xacro" params="xyz">
         <!-- =========== 相机模块==================-->
@@ -13,4 +14,14 @@
                 </material>
             </visual>
+            <collision>
+                <origin xyz="0 0 0" rpy="0 0 0" />
+                <geometry>
+                    <box size="0.02 0.1 0.02" />
+                </geometry>
+                <material name="green">
+                    <color rgba="0.0 1.0 0.0 0.8" />
+                </material>
+            </collision>
+            <xacro:box_inertia m="0.01" w="0.02" h="0.10" d="0.02" />
         </link>
         <joint name="camera_joint" type="fixed">
@@ -19,4 +30,7 @@
             <origin xyz="${xyz}" />
         </joint>
+        <gazebo reference="camera_link">
+            <material>Gazebo/Green</material>
+        </gazebo>
     </xacro:macro>
 </robot>

File: src/robot_description/urdf/fishbot/sensor/imu.urdf.xacro (robot description, xacro)
@@ -1,4 +1,5 @@
 <?xml version="1.0"?>
 <robot xmlns:xacro="http://www.ros.org/wiki/xacro">
+    <xacro:include filename="$(find robot_description)/urdf/fishbot/common_inertia.xacro" />
     <xacro:macro name="imu_xacro" params="xyz">
         <link name="imu_link">
@@ -12,4 +13,14 @@
                 </material>
             </visual>
+            <collision>
+                <origin xyz="0 0 0" rpy="0 0 0" />
+                <geometry>
+                    <box size="0.02 0.02 0.02" />
+                </geometry>
+                <material name="black">
+                    <color rgba="0.0 0.0 0.0 0.8" />
+                </material>
+            </collision>
+            <xacro:box_inertia m="0.01" w="0.02" h="0.02"  d="0.02" />
         </link>
         <joint name="imu_joint" type="fixed">

File: src/robot_description/urdf/fishbot/sensor/laser.urdf.xacro (robot description, xacro)
@@ -1,4 +1,5 @@
 <?xml version="1.0"?>
 <robot xmlns:xacro="http://www.ros.org/wiki/xacro">
+    <xacro:include filename="$(find robot_description)/urdf/fishbot/common_inertia.xacro" />
     <xacro:macro name="laser_xacro" params="xyz">
         <!-- ================== 雷达支撑杆====================== -->
@@ -13,4 +14,14 @@
                 </material>
             </visual>
+            <collision>
+                <origin xyz="0 0 0" rpy="0 0 0" />
+                <geometry>
+                    <cylinder length="0.10" radius="0.01" />
+                </geometry>
+                <material name="green">
+                    <color rgba="0.0 1.0 0.0 0.8" />
+                </material>
+            </collision>
+            <xacro:cylinder_inertia m="1.0" r="0.01" h="0.10" />
         </link>
         <joint name="laser_cylinder_joint" type="fixed">
@@ -30,4 +41,14 @@
                 </material>
             </visual>
+            <collision>
+                <origin xyz="0 0 0" rpy="0 0 0" />
+                <geometry>
+                    <cylinder length="0.02" radius="0.02" />
+                </geometry>
+                <material name="green">
+                    <color rgba="0.0 1.0 0.0 0.8" />
+                </material>
+            </collision>
+            <xacro:cylinder_inertia m="0.03" r="0.02" h="0.02" />
         </link>
         <joint name="laser_joint" type="fixed">
@@ -36,4 +57,10 @@
             <origin xyz="0 0 0.05" />
         </joint>
+        <gazebo reference="laser_cylinder_link">
+            <material>Gazebo/Black</material>
+        </gazebo>
+        <gazebo reference="laser_link">
+            <material>Gazebo/Black</material>
+        </gazebo>
     </xacro:macro>
 </robot>
